File: hardware/USB_glitcher.kicad_pcb (KiCad board)
At the start: 2 copper layers, 52.6 x 46.2 mm, 32 parts, among them Q1 NPN, Q2 IRLML6302, SW1 SWITCH, U1 MCP1700, U2 MAX4619

Commit message: PCB v.0.2 + Fix Vcc MAX4619. + Fix layout for testpoint. + Fix SWDIO and USB pin mapping. + Fix resistor divider before NPN transistor.
Parts:
- moved R7 2.95 mm to (170.2, 91.2)
- moved R5 2.78 mm to (168.2, 91.2)
Connections:
- DD1 pad 12: Net-(DD1-Pad12) -> (no net)
- DD1 pad 13: Net-(DD1-Pad13) -> (no net)
- DD1 pad 18: Net-(DD1-Pad18) -> (no net)
- DD1 pad 2: Net-(DD1-Pad2) -> (no net)
- DD1 pad 20: Net-(DD1-Pad20) -> (no net)
- DD1 pad 21: Net-(DD1-Pad21) -> /USB_DM
- DD1 pad 22: /USB_DM -> /USB_DP
- DD1 pad 23: /USB_DP -> /SWDIO
- DD1 pad 24: /SWDIO -> /SWCLK
- DD1 pad 25: /SWCLK -> (no net)
- DD1 pad 27: Net-(DD1-Pad27) -> (no net)
- DD1 pad 28: Net-(DD1-Pad28) -> (no net)
- DD1 pad 3: Net-(DD1-Pad3) -> (no net)
- DD1 pad 32: Net-(DD1-Pad32) -> (no net)
- DD1 pad 4: Net-(DD1-Pad4) -> (no net)
- DD1 pad 6: Net-(DD1-Pad6) -> (no net)
- R7 pad 1: +3.3V -> /LED
- R7 pad 2: /LED -> GND
- U2 pad 16: +3.3V -> +5V
Routing:
- net +5V: track 9.89 -> 51.7 mm, vias 0 -> 2
- net +3.3V: track 114.4 -> 85.1 mm
- net GND: track 223.5 -> 226.0 mm
- net /SWCLK: track 32.1 -> 30.3 mm
- net /DEVICE_POWER_EN: track 23.5 -> 22.2 mm
- net /LED: track 22.6 -> 23.9 mm
Other:
- board text added: "@RL USB_glitcher v.0.2"
- board text removed: "@RL USB_glitcher v.0.1"
