File: hardware/USB_glitcher.sch (KiCad schematic (older format))
At the start: 32 parts, among them Q1 NPN, Q2 IRLML6302, SW1 SWITCH, U1 MCP1700, U2 MAX4619

Commit message: PCB v.0.2 + Fix Vcc MAX4619. + Fix layout for testpoint. + Fix SWDIO and USB pin mapping. + Fix resistor divider before NPN transistor.
Parts:
- C1, C2, C3, C4, C5, C6, C7: symbol C -> Tittar_kl:C
- D1: symbol LED -> Tittar_kl:LED
- DD1: symbol STM32F050K4_6 -> st_kl:STM32F050K4_6
- Q1: symbol NPN -> Transistors_kl:NPN
- Q2: symbol IRLML6302 -> Transistors_kl:IRLML6302
- R1, R2, R3, R4, R5, R6, R7, R8: symbol R -> Tittar_kl:R
- SW1: symbol SWITCH -> Tittar_kl:SWITCH
- TP1, TP2: footprint Connectors:PLS-1Rnd -> Connectors:Round_1MM5; symbol TESTPOINT -> pcb_details:TESTPOINT
- U1: symbol MCP1700 -> Power_kl:MCP1700
- U2: symbol MAX4619 -> Switches:MAX4619
- XL1: symbol CONN_8 -> Connectors_kl:CONN_8
- XL2, XL3, XL4: symbol CONN_2 -> Connectors_kl:CONN_2
- XL5: symbol ST_SWD -> Connectors_kl:ST_SWD
- XL6, XL7: symbol USB_A -> Connectors_kl:USB_A
- XL8: symbol USB_B -> Connectors_kl:USB_B
Connections:
- wire segments 131 -> 153
